File: Sensing/Sensor_Breakouts/MEu-2CO_breakout/MEu-2CO.kicad_pcb (KiCad board)
At the start: 2 copper layers, 30.5 x 20.2 mm, 8 parts, among them J1 Conn_01x03_Pin, U1 MEu-2CO, U2 LT6003HS5TRPBF

Commit message: Added Hydrogen sensor and modified pins
I created a PCB and schematic for the hydrogen sensor. I also changed the footprints to allow for quick component insertion
Routing:
- net +5V: track 28.7 -> 29.7 mm
Changed lines of the file:
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@@
 		(pad "1" thru_hole circle
 			(at -6.75 0)
-			(size 3 3)
-			(drill 2)
+			(size 3.7 3.7)
+			(drill 2.7)
 			(layers "*.Cu" "*.Mask")
 			(remove_unused_layers no)
@@
 		(pad "2" thru_hole circle
 			(at 0 -6.75)
-			(size 3 3)
-			(drill 2)
+			(size 3.7 3.7)
+			(drill 2.7)
 			(layers "*.Cu" "*.Mask")
 			(remove_unused_layers no)
@@
 	)
 	(segment
-		(start 110.221999 114.3)
-		(end 105.2 114.3)
-		(width 0.2)
-		(layer "F.Cu")
-		(net 3)
-	)
-	(segment
-		(start 111.951 120.549)
-		(end 111.951 116.029001)
+		(start 106.5 126)
+		(end 112.5 120)
 		(width 0.2)
 		(layer "F.Cu")
@@
 	)
 	(segment
-		(start 106.5 126)
-		(end 111.951 120.549)
+		(start 111.05 114.3)
+		(end 105.2 114.3)
+		(width 0.2)
+		(layer "F.Cu")
+		(net 3)
+	)
+	(segment
+		(start 112.5 120)
+		(end 112.5 115.75)
 		(width 0.2)
 		(layer "F.Cu")
@@
 	)
 	(segment
-		(start 111.951 116.029001)
-		(end 110.221999 114.3)
-		(width 0.2)
-		(layer "F.Cu")
+		(start 112.5 115.75)
+		(end 111.05 114.3)
+		(width 0.2)
+		(layer "F.Cu")

Commit message: Made small CO PCB changes
Routing:
- net Net-(U2-OUT): track 13.2 -> 14.7 mm
Other:
- board text added: "+5V"
- board text added: "Gnd"
- board text added: "V_{out}"
